File: pcb/stepperDriver.kicad_pcb (KiCad board)
At the start: 2 copper layers, 18 parts, among them IC1 ATTINY84-P, P1 CONN_6, P2 CONN_7, U1 L298D

Commit message: axeXY
Routing:
- added copper zone on B.Cu, net GND
- added copper zone on B.Cu, net N-0000019
Changed lines of the file:
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@@
-(kicad_pcb (version 3) (host pcbnew "(2013-05-16 BZR 4016)-stable")
+(kicad_pcb (version 3) (host pcbnew "(2013-05-31 BZR 4019)-stable")
   (general
     (links 51)
     (no_connects 0)
-    (area 50.749999 44.399999 109.270001 86.410001)
+    (area 50.393599 44.399999 109.270001 86.410001)
     (thickness 1.6)
     (drawings 4)
@@
   )
   (setup
-    (last_trace_width 1)
+    (last_trace_width 0.8)
     (user_trace_width 0.5)
+    (user_trace_width 0.8)
     (user_trace_width 1)
     (trace_clearance 0.254)
@@
     (pad_to_mask_clearance 0)
     (aux_axis_origin 0 0)
-    (visible_elements FFFFFFBF)
+    (visible_elements 7FFFFFFF)
     (pcbplotparams
       (layerselection 3178497)
@@
   (segment (start 59.69 80.01) (end 59.69 80.01) (width 0.5) (layer Dessous.Cu) (net 1) (status 80000))
   (segment (start 59.69 80.01) (end 59.69 74.93) (width 0.5) (layer Dessous.Cu) (net 1) (status 80000))
-  (segment (start 83.82 82.55) (end 85.09 82.55) (width 1) (layer Dessous.Cu) (net 2) (status 400000))
-  (segment (start 85.09 80.01) (end 85.09 82.55) (width 1) (layer Dessous.Cu) (net 2) (status 400000))
+  (segment (start 83.82 82.55) (end 85.09 82.55) (width 1) (layer Dessous.Cu) (net 2))
+  (segment (start 85.09 80.01) (end 85.09 82.55) (width 1) (layer Dessous.Cu) (net 2))
   (segment (start 85.09 82.55) (end 85.09 85.09) (width 1) (layer Dessous.Cu) (net 2))
   (segment (start 90.17 85.09) (end 90.17 81.28) (width 1) (layer Dessous.Cu) (net 2))
@@
   (segment (start 73.66 63.5) (end 73.66 69.85) (width 0.5) (layer Dessous.Cu) (net 9))
   (segment (start 76.2 60.96) (end 73.66 63.5) (width 0.5) (layer Dessous.Cu) (net 9))
-  (segment (start 80.01 62.23) (end 85.09 62.23) (width 1) (layer Dessous.Cu) (net 10) (status 800000))
+  (segment (start 80.01 62.23) (end 85.09 62.23) (width 1) (layer Dessous.Cu) (net 10))
   (segment (start 80.01 62.23) (end 80.01 58.42) (width 1) (layer Dessous.Cu) (net 10))
   (segment (start 76.2 77.47) (end 76.2 76.2) (width 0.5) (layer Dessous.Cu) (net 10))
@@
   (segment (start 100.33 49.53) (end 100.33 46.99) (width 1) (layer Dessous.Cu) (net 12))
   (segment (start 66.04 53.34) (end 63.5 55.88) (width 1) (layer Dessous.Cu) (net 12))
-  (segment (start 82.55 46.99) (end 85.09 49.53) (width 1) (layer Dessous.Cu) (net 12))
-  (segment (start 62.23 46.99) (end 82.55 46.99) (width 1) (layer Dessous.Cu) (net 12))
+  (segment (start 82.55 46.99) (end 85.09 49.53) (width 0.8) (layer Dessous.Cu) (net 12))
+  (segment (start 62.23 46.99) (end 82.55 46.99) (width 0.8) (layer Dessous.Cu) (net 12))
   (segment (start 82.55 46.99) (end 82.55 46.99) (width 0.5) (layer Dessous.Cu) (net 12))
-  (segment (start 60.96 48.26) (end 62.23 46.99) (width 1) (layer Dessous.Cu) (net 12))
-  (segment (start 60.96 54.61) (end 60.96 48.26) (width 1) (layer Dessous.Cu) (net 12))
+  (segment (start 60.96 48.26) (end 62.23 46.99) (width 0.8) (layer Dessous.Cu) (net 12))
+  (segment (start 60.96 54.61) (end 60.96 48.26) (width 0.8) (layer Dessous.Cu) (net 12))
   (segment (start 62.23 55.88) (end 60.96 54.61) (width 1) (layer Dessous.Cu) (net 12))
   (segment (start 63.5 55.88) (end 62.23 55.88) (width 1) (layer Dessous.Cu) (net 12))
   (segment (start 97.79 46.99) (end 97.79 49.53) (width 1) (layer Dessous.Cu) (net 12))
-  (segment (start 85.09 49.53) (end 97.79 49.53) (width 1) (layer Dessous.Cu) (net 12))
+  (segment (start 85.09 49.53) (end 97.79 49.53) (width 0.8) (layer Dessous.Cu) (net 12))
   (segment (start 107.95 49.53) (end 105.41 49.53) (width 1) (layer Dessous.Cu) (net 12))
   (segment (start 105.41 49.53) (end 102.87 49.53) (width 1) (layer Dessous.Cu) (net 12))
@@
   (segment (start 105.41 57.15) (end 105.41 59.69) (width 1) (layer Dessous.Cu) (net 14))
   (segment (start 102.87 54.61) (end 105.41 57.15) (width 1) (layer Dessous.Cu) (net 14))
-  (segment (start 87.63 54.61) (end 102.87 54.61) (width 1) (layer Dessous.Cu) (net 14))
-  (segment (start 81.28 48.26) (end 87.63 54.61) (width 1) (layer Dessous.Cu) (net 14))
-  (segment (start 66.04 48.26) (end 81.28 48.26) (width 1) (layer Dessous.Cu) (net 14))
-  (segment (start 63.5 50.8) (end 66.04 48.26) (width 1) (layer Dessous.Cu) (net 14))
+  (segment (start 87.63 54.61) (end 102.87 54.61) (width 0.8) (layer Dessous.Cu) (net 14))
+  (segment (start 81.28 48.26) (end 87.63 54.61) (width 0.8) (layer Dessous.Cu) (net 14))
+  (segment (start 66.04 48.26) (end 81.28 48.26) (width 0.8) (layer Dessous.Cu) (net 14))
+  (segment (start 63.5 50.8) (end 66.04 48.26) (width 0.8) (layer Dessous.Cu) (net 14))
   (segment (start 105.41 64.77) (end 105.41 69.85) (width 1) (layer Dessous.Cu) (net 14) (status 80000))
   (segment (start 105.41 59.69) (end 105.41 64.77) (width 1) (layer Dessous.Cu) (net 14) (status 80000))
@@
   (segment (start 102.87 57.15) (end 102.87 59.69) (width 1) (layer Dessous.Cu) (net 15))
   (segment (start 101.6 55.88) (end 102.87 57.15) (width 1) (layer Dessous.Cu) (net 15))
-  (segment (start 86.36 55.88) (end 101.6 55.88) (width 1) (layer Dessous.Cu) (net 15))
-  (segment (start 67.31 50.8) (end 68.58 49.53) (width 1) (layer Dessous.Cu) (net 15))
+  (segment (start 86.36 55.88) (end 101.6 55.88) (width 0.8) (layer Dessous.Cu) (net 15))
+  (segment (start 67.31 50.8) (end 68.58 49.53) (width 0.8) (layer Dessous.Cu) (net 15))
   (segment (start 67.31 54.61) (end 67.31 52.07) (width 0.5) (layer Dessous.Cu) (net 15))
   (segment (start 67.31 52.07) (end 67.31 50.8) (width 1) (layer Dessous.Cu) (net 15))
@@
   (segment (start 102.87 59.69) (end 102.87 64.77) (width 1) (layer Dessous.Cu) (net 15) (status 80000))
   (segment (start 102.87 64.77) (end 102.87 69.85) (width 1) (layer Dessous.Cu) (net 15) (status 80000))
-  (segment (start 80.01 49.53) (end 86.36 55.88) (width 1) (layer Dessous.Cu) (net 15))
-  (segment (start 68.58 49.53) (end 80.01 49.53) (width 1) (layer Dessous.Cu) (net 15))
+  (segment (start 80.01 49.53) (end 86.36 55.88) (width 0.8) (layer Dessous.Cu) (net 15))
+  (segment (start 68.58 49.53) (end 80.01 49.53) (width 0.8) (layer Dessous.Cu) (net 15))
   (segment (start 77.47 58.42) (end 77.47 57.15) (width 1) (layer Dessous.Cu) (net 16))
   (segment (start 85.09 59.69) (end 97.79 59.69) (width 1) (layer Dessous.Cu) (net 16))
@@
   (segment (start 66.04 69.85) (end 66.04 66.04) (width 0.5) (layer Dessous.Cu) (net 18) (status 80000))
   (segment (start 78.74 77.47) (end 78.74 82.55) (width 0.5) (layer Dessous.Cu) (net 19) (status 80000))
+  (zone (net 12) (net_name N-0000019) (layer Dessous.Cu) (hatch edge 0.508)
+    (connect_pads (clearance 0.508))
+    (min_thickness 0.254)
+    (fill (arc_segments 16) (thermal_gap 0.508) (thermal_bridge_width 0.508))
+    (polygon
+      (pts
+        (xy 109.22 73.66) (xy 96.52 73.66) (xy 96.52 54.61) (xy 60.96 53.34) (xy 60.96 62.23)
+        (xy 50.8 62.23) (xy 50.8 44.45) (xy 109.22 44.45)
+      )
+    )
+  )
+  (zone (net 2) (net_name GND) (layer Dessous.Cu) (hatch edge 0.508)
+    (connect_pads (clearance 0.508))
+    (min_thickness 0.254)
+    (fill (arc_segments 16) (thermal_gap 0.508) (thermal_bridge_width 0.508))
+    (polygon
+      (pts
+        (xy 109.22 86.36) (xy 50.8 86.36) (xy 50.8 63.5) (xy 62.23 63.5) (xy 62.23 54.61)
+        (xy 63.5 55.88) (xy 95.25 55.88) (xy 95.25 74.93) (xy 109.22 74.93)
+      )
+    )
+  )
 )
