File: pcb/optoSwitch/optoSwitch.sch (KiCad schematic (older format))
At the start: 4 parts, among them IC1 OPTOSWITCH, K1 CONN_3

Commit message: Correction résistance pullup
Parts:
- R2: value 2k2 -> 4k7
Changed lines of the file:
@@
-EESchema Schematic File Version 2  date 15.06.2013 17:59:46
+EESchema Schematic File Version 2  date 27.06.2013 12:45:07
 LIBS:marcha
 LIBS:power
@@
 LIBS:contrib
 LIBS:valves
+LIBS:optoSwitch-cache
 EELAYER 27 0
 EELAYER END
@@
 Sheet 1 1
 Title ""
-Date "15 jun 2013"
+Date "27 jun 2013"
 Rev ""
 Comp ""
@@
 P 4200 2400
 F 0 "R2" V 4280 2400 40  0000 C CNN
-F 1 "2k2" V 4207 2401 40  0000 C CNN
+F 1 "4k7" V 4207 2401 40  0000 C CNN
 F 2 "~" V 4130 2400 30  0000 C CNN
 F 3 "~" H 4200 2400 30  0000 C CNN
